Commit message: depth cam

File: jackal_ws/src/jackal/jackal_description/urdf/jackal.urdf.xacro (robot description, xacro)
@@ -245,5 +245,5 @@
       <origin xyz="0 0 0" rpy="0 0 0"/>
       <geometry>
-    <box size="${camera_link} ${camera_link} ${camera_link}"/>
+        <box size="${camera_link} ${camera_link} ${camera_link}"/>
       </geometry>
     </collision>
@@ -251,5 +251,5 @@
       <origin xyz="0 0 0" rpy="0 0 0"/>
       <geometry>
-    <box size="${camera_link} ${camera_link} ${camera_link}"/>
+        <box size="${camera_link} ${camera_link} ${camera_link}"/>
       </geometry>
       <material name="black"/>

File: jackal_ws/src/jackal_3dmain/urdf/jackal.gazebo.xacro (robot description, xacro)
@@ -81,5 +81,5 @@
     <!-- Camera -->
     <gazebo reference="${frame_prefix}camera_link">
-      <sensor type="camera" name="camera">
+      <sensor type="depth" name="camera">
         <update_rate>${cameraRate}</update_rate>
         <camera name="head">
@@ -103,20 +103,30 @@
           </noise>
         </camera>
-        <plugin name="camera_controller" filename="libgazebo_ros_camera.so">
+        <plugin name="camera_plugin" filename="libgazebo_ros_openni_kinect.so">
+          <robotNamespace>${robot_name}</robotNamespace>
+          <baseline>0.2</baseline>
           <alwaysOn>true</alwaysOn>
+          <!-- Keep this zero, update_rate in the parent <sensor> tag
+            will control the frame rate. -->
           <updateRate>0.0</updateRate>
-          <cameraName>camera</cameraName>
-          <imageTopicName>${topic_prefix}image_raw</imageTopicName>
-          <cameraInfoTopicName>${topic_prefix}camera_info</cameraInfoTopicName>
-          <frameName>${frame_prefix}camera_link</frameName>
-          <!-- setting hackBaseline to anything but 0.0 will cause a misalignment
-            between the gazebo sensor image and the frame it is supposed to
-            be attached to -->
-          <hackBaseline>0.0</hackBaseline>
-          <distortionK1>0.0</distortionK1>
-          <distortionK2>0.0</distortionK2>
-          <distortionK3>0.0</distortionK3>
-          <distortionT1>0.0</distortionT1>
-          <distortionT2>0.0</distortionT2>
+          <cameraName>camera_ir</cameraName>
+          <imageTopicName>/camera/color/image_raw</imageTopicName>
+          <cameraInfoTopicName>/camera/color/camera_info</cameraInfoTopicName>
+          <depthImageTopicName>/camera/depth/image_raw</depthImageTopicName>
+          <depthImageCameraInfoTopicName>/camera/depth/camera_info</depthImageCameraInfoTopicName>
+          <pointCloudTopicName>/camera/depth/points</pointCloudTopicName>
+          <frameName>camera_link</frameName>
+          <pointCloudCutoff>0.5</pointCloudCutoff>
+          <pointCloudCutoffMax>3.0</pointCloudCutoffMax>
+          <distortionK1>0</distortionK1>
+          <distortionK2>0</distortionK2>
+          <distortionK3>0</distortionK3>
+          <distortionT1>0</distortionT1>
+          <distortionT2>0</distortionT2>
+          <CxPrime>0</CxPrime>
+          <Cx>0</Cx>
+          <Cy>0</Cy>
+          <focalLength>0</focalLength>
+          <hackBaseline>0</hackBaseline>
         </plugin>
       </sensor>
