Commit message: Camera fix and LLM (requires socket)

File: jackal_ws/src/jackal_3dmain/urdf/jackal.gazebo.xacro (robot description, xacro)
@@ -1,5 +1,5 @@
 <?xml version="1.0"?>
 <robot name="jackal_gazebo" xmlns:xacro="http://www.ros.org/wiki/xacro">
-  <xacro:macro name="jackal_gazebo" params="name frame_prefix topic_prefix imuRate:=100 cameraRate:=30">
+  <xacro:macro name="jackal_gazebo" params="name frame_prefix topic_prefix imuRate:=100 cameraRate:=30 ">
     <!-- different management if we don't want multiple robots -->
     <xacro:if value="${(frame_prefix == '')}">
@@ -104,5 +104,5 @@
         </camera>
         <plugin name="camera_plugin" filename="libgazebo_ros_openni_kinect.so">
-          <robotNamespace>${robot_name}</robotNamespace>
+          <robotNamespace>${name}</robotNamespace>
           <baseline>0.2</baseline>
           <alwaysOn>true</alwaysOn>
@@ -110,10 +110,10 @@
             will control the frame rate. -->
           <updateRate>0.0</updateRate>
-          <cameraName>camera_ir</cameraName>
-          <imageTopicName>/camera/color/image_raw</imageTopicName>
-          <cameraInfoTopicName>/camera/color/camera_info</cameraInfoTopicName>
-          <depthImageTopicName>/camera/depth/image_raw</depthImageTopicName>
-          <depthImageCameraInfoTopicName>/camera/depth/camera_info</depthImageCameraInfoTopicName>
-          <pointCloudTopicName>/camera/depth/points</pointCloudTopicName>
+          <cameraName>/</cameraName>
+          <imageTopicName>camera/image_raw</imageTopicName>
+          <cameraInfoTopicName>camera/camera_info</cameraInfoTopicName>
+          <depthImageTopicName>camera/depth/image_raw</depthImageTopicName>
+          <depthImageCameraInfoTopicName>camera/depth/camera_info</depthImageCameraInfoTopicName>
+          <pointCloudTopicName>camera/depth/points</pointCloudTopicName>
           <frameName>camera_link</frameName>
           <pointCloudCutoff>0.5</pointCloudCutoff>
